File: Fase3/PCBs/Estacao/Estacao.kicad_pcb (KiCad board)
At the start: 2 copper layers, 104.1 x 97.8 mm, 31 parts, among them J1 WCM, J2 I2C, J3 I2C, J4 Conn_01x02, J5 GPS, J6 I2C, SW2 SW_Wuerth_450301014042, SW3 SW_Wuerth_450301014042, SW4 SW_Push, SW5 SW_Push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

Commit message: Updade Slik da PCB V01
Parts:
- added ?: , , F.Cu at (194.3, 128.3)
- added TP1: GND, Connector_PinHeader_2.54mm:PinHeader_1x01_P2.54mm_Vertical, F.Cu at (172.7, 43.2)
- A1: value RaspberryPi_Pico -> Raspberry Pi Pico
- BT1: value Battery_Cell -> Battery
- D1: renamed from D3; value LED -> G
- D2: value LED -> B
- D3: renamed from D1; value LED -> R
- Dc-Dc1: value ~ -> 20V to 5V
- J1: footprint Connector_Molex:Molex_SL_171971-0006_1x06_P2.54mm_Vertical -> Connector_PinSocket_2.54mm:PinSocket_1x06_P2.54mm_Vertical
- J2: value I2C -> I2C-1; footprint Connector_JST:JST_EH_B4B-EH-A_1x04_P2.50mm_Vertical -> Connector_JST:JST_XH_B4B-XH-A_1x04_P2.50mm_Vertical
- J3: value I2C -> I2C-2; footprint Connector_JST:JST_EH_B4B-EH-A_1x04_P2.50mm_Vertical -> Connector_JST:JST_XH_B4B-XH-A_1x04_P2.50mm_Vertical
- J4: renamed from J6; value I2C -> I2C-3; footprint Connector_JST:JST_EH_B4B-EH-A_1x04_P2.50mm_Vertical -> Connector_JST:JST_XH_B4B-XH-A_1x04_P2.50mm_Vertical
- J5: footprint Connector_JST:JST_EH_B4B-EH-A_1x04_P2.50mm_Vertical -> Connector_JST:JST_XH_B4B-XH-A_1x04_P2.50mm_Vertical
- J6: renamed from J4; value Conn_01x02 -> Photo Cel; footprint TerminalBlock:TerminalBlock_Altech_AK300-2_P5.00mm -> Connector_Molex:Molex_SL_171971-0002_1x02_P2.54mm_Vertical
- SW1: renamed from SW2; footprint Button_Switch_THT:SW_Slide-03_Wuerth-WS-SLTV_10x2.5x6.4_P2.54mm -> PcbLibrary:switch_3p_2mm
- SW2: renamed from SW6; footprint Button_Switch_THT:SW_Slide-03_Wuerth-WS-SLTV_10x2.5x6.4_P2.54mm -> PcbLibrary:switch_3p_2mm
- SW3: footprint Button_Switch_THT:SW_Slide-03_Wuerth-WS-SLTV_10x2.5x6.4_P2.54mm -> PcbLibrary:switch_3p_2mm
- SW4: value SW_Push -> Config
- SW5: value SW_Push -> Reset
- moved REF** 12.8 mm to (97.8, 128.3)
- moved BT1 4.14 mm to (182.9, 122.6)
- moved SW3 3.85 mm to (147.9, 43.2), turned to 0 degrees
- moved J2 3.54 mm to (108.0, 59.7)
- moved J1 2.54 mm to (105.4, 49.5), turned to 90 degrees
- moved REF** 1.80 mm to (194.3, 38.1)
- moved REF** 1.80 mm to (97.8, 38.1)
- moved J3 1.77 mm to (108.0, 67.3)
- moved SW2 1.46 mm to (183.4, 41.9), turned to 0 degrees
- moved SW1 1.46 mm to (142.2, 123.7), turned to -90 degrees
- moved SW4 1.27 mm to (115.0, 87.3)
- moved SW5 1.27 mm to (115.0, 105.4)
- moved C2 1.27 mm to (156.2, 52.1)
- moved C3 1.27 mm to (166.4, 52.1)
- moved J4 0.08 mm to (108.0, 74.9)
Connections:
- SW3 pad 1: Net-(A1-VSYS) -> Net-(D4-K)
- SW3 pad 2: Net-(A1-VSYS) -> Net-(D4-K)
- SW3 pad 3: Net-(D4-K) -> Net-(A1-VSYS)
Routing:
- net Net-(A1-GPIO3): track 36.4 -> 44.1 mm
- net Net-(A1-GPIO2): track 39.7 -> 47.4 mm
- net Net-(D4-K): track 12.5 -> 7.08 mm
- net GND: track 11.7 -> 15.3 mm
- net Net-(A1-3V3): track 187.1 -> 190.5 mm
- net Net-(BT1--): track 44.7 -> 47.9 mm
- net Net-(A1-VSYS): track 37.7 -> 40.8 mm
- net Net-(A1-GPIO0): track 21.2 -> 23.7 mm
- net Net-(A1-GPIO1): track 25.5 -> 28.0 mm
- net Net-(BT1-+): track 92.6 -> 91.0 mm
- net Net-(A1-RUN): track 40.5 -> 39.2 mm
- net Net-(A1-GPIO5): track 19.4 -> 18.2 mm
- net Net-(J6-Pin_2): track 8.15 -> 9.41 mm
- net Net-(Charger1-Bat+): track 72.1 -> 72.6 mm
Other:
- board text added: "- +"
- board text added: "3V3"
- board text added: "Estação Meteorológica V 01"
- board text added: "GND"
- board text added: "RX"
- board text added: "TX"
