File: Fase3/PCBs/Estacao/Estacao.kicad_sch (KiCad schematic)
At the start: 28 parts, among them J1 WCM, J2 I2C, J3 I2C, J4 Conn_01x02, J5 GPS, J6 I2C, SW2 SW_Wuerth_450301014042, SW3 SW_Wuerth_450301014042, SW4 SW_Push, SW5 SW_Push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

Commit message: Updade Slik da PCB V01
Parts:
- added TP1: GND, Connector_PinHeader_2.54mm:PinHeader_1x01_P2.54mm_Vertical, symbol Connector:TestPoint
- A1: value RaspberryPi_Pico -> Raspberry Pi Pico
- BT1: value Battery_Cell -> Battery
- D1: renamed from D3; value LED -> G
- D2: value LED -> B
- D3: renamed from D1; value LED -> R
- Dc-Dc1: value ~ -> 20V to 5V
- J1: footprint Connector_Molex:Molex_SL_171971-0006_1x06_P2.54mm_Vertical -> Connector_PinSocket_2.54mm:PinSocket_1x06_P2.54mm_Vertical
- J2: value I2C -> I2C-1; footprint Connector_JST:JST_EH_B4B-EH-A_1x04_P2.50mm_Vertical -> Connector_JST:JST_XH_B4B-XH-A_1x04_P2.50mm_Vertical
- J3: value I2C -> I2C-2; footprint Connector_JST:JST_EH_B4B-EH-A_1x04_P2.50mm_Vertical -> Connector_JST:JST_XH_B4B-XH-A_1x04_P2.50mm_Vertical
- J4: renamed from J6; value I2C -> I2C-3; footprint Connector_JST:JST_EH_B4B-EH-A_1x04_P2.50mm_Vertical -> Connector_JST:JST_XH_B4B-XH-A_1x04_P2.50mm_Vertical
- J5: footprint Connector_JST:JST_EH_B4B-EH-A_1x04_P2.50mm_Vertical -> Connector_JST:JST_XH_B4B-XH-A_1x04_P2.50mm_Vertical
- J6: renamed from J4; value Conn_01x02 -> Photo Cel; footprint TerminalBlock:TerminalBlock_Altech_AK300-2_P5.00mm -> Connector_Molex:Molex_SL_171971-0002_1x02_P2.54mm_Vertical
- SW1: renamed from SW2; footprint Button_Switch_THT:SW_Slide-03_Wuerth-WS-SLTV_10x2.5x6.4_P2.54mm -> PcbLibrary:switch_3p_2mm
- SW2: renamed from SW6; footprint Button_Switch_THT:SW_Slide-03_Wuerth-WS-SLTV_10x2.5x6.4_P2.54mm -> PcbLibrary:switch_3p_2mm
- SW3: footprint Button_Switch_THT:SW_Slide-03_Wuerth-WS-SLTV_10x2.5x6.4_P2.54mm -> PcbLibrary:switch_3p_2mm
- SW4: value SW_Push -> Config
- SW5: value SW_Push -> Reset
Connections:
- net GND: now also TP1.1
- net at A1.39 (VSYS), C2.1, R5.1: now also SW3.3 (A); no longer SW3.1 (B), SW3.2 (C)
- net at D4.1 (K): now also SW3.1 (B), SW3.2 (C); no longer SW3.3 (A)
Other:
- moved on the sheet: SW3
