File: Fase3/Hardware/Estacao/Estacao.kicad_sch (KiCad schematic)
At the start: 29 parts, among them J1 WCM, J2 I2C-1, J3 I2C-2, J4 I2C-3, J5 GPS, J6 Photo Cel, SW1 SW_Wuerth_450301014042, SW2 SW_Wuerth_450301014042, SW3 SW_Wuerth_450301014042, SW4 Config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

Commit message: Update PCB V03
Parts:
- removed SW1, SW2, SW3: SW_Wuerth_450301014042, PcbLibrary:switch_3p_2mm, symbol Switch:SW_Wuerth_450301014042
- added D5: 1N5819, Diode_THT:D_DO-41_SOD81_P10.16mm_Horizontal, symbol Diode:1N5819
- added SW1, SW2, SW3: SW_SPDT, PcbLibrary:switch_3p_2mm_e_2.54mm, symbol Switch:SW_SPDT
- BT1: value Battery -> Battery 18650 2000mAh; footprint Battery:BatteryHolder_MPD_BK-18650-PC2 -> PcbLibrary:BatteryHolder_MPD_BK-18650-PC2b
- C3: value C_Polarized -> 100 uF
- C4: value C -> 100n
- Charger1: value ~ -> HW-107
- Dc-Dc1: value 20V to 5V -> LN2596 DC-DC HW-411 21V to 5V
- J6: footprint Connector_Molex:Molex_SL_171971-0002_1x02_P2.54mm_Vertical -> PcbLibrary:Molex_SL_171971-0002_1x02_P2.54mm_Vertical_b
- R1, R2, R3: value R -> 1k
- R4, R5: value R -> 100k
Connections:
- net GND: now also A1.33 (AGND)
- net at C3.1, Charger1.4 (Bat+): now also SW2.1 (A)
- net at J6.2 (Pin_2): now also D5.2 (A)
- net at A1.39 (VSYS), C2.1, R5.1: now also SW3.1 (A)
- net at D4.1 (K): now also SW3.2 (B), SW3.3 (C)
- net at BT1.1 (+): now also SW2.2 (B), SW2.3 (C)
- net at Dc-Dc1.1 (IN+): now also SW1.2 (B), SW1.3 (C)
- new net: D5.1 (K), SW1.1 (A)
Other:
- company: (none) -> Embarcatech / Feec
- title: (none) -> Estação Meteorológica
- moved on the sheet: BT1, J6

Commit message: UpdatePcb V3
Parts:
- C1, C2, C3: footprint Capacitor_THT:CP_Radial_D8.0mm_P3.50mm -> Capacitor_THT:CP_Radial_D7.5mm_P2.50mm
- J6: footprint PcbLibrary:Molex_SL_171971-0002_1x02_P2.54mm_Vertical_b -> PcbLibrary:BorneBatSolar
- SW1, SW2, SW3: footprint PcbLibrary:switch_3p_2mm_e_2.54mm -> PcbLibrary:switch_3p_2.54mm_on_off
Connections:
- net at J6.1 (Pin_1): now also D5.2 (A); no longer Dc-Dc1.2 (IN-)
- net at J6.2 (Pin_2): now also Dc-Dc1.2 (IN-); no longer D5.2 (A)
- net at A1.1 (GPIO0): now also J1.2 (Pin_2); no longer J1.3 (Pin_3)
- net at A1.2 (GPIO1): now also J1.3 (Pin_3); no longer J1.2 (Pin_2)
Other:
- moved on the sheet: J6
Changed lines of the file:
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@@
 	(wire
 		(pts
+			(xy 33.02 146.05) (xy 35.56 146.05)
+		)
+		(stroke
+			(width 0)
+			(type default)
+		)
+	)
+	(wire
+		(pts
 			(xy 146.05 21.59) (xy 146.05 29.21)
 		)
@@
 	(wire
 		(pts
-			(xy 177.8 80.01) (xy 161.29 80.01)
-		)
-		(stroke
-			(width 0)
-			(type default)
-		)
-	)
-	(wire
-		(pts
 			(xy 115.57 123.19) (xy 115.57 120.65)
 		)
@@
 	(wire
 		(pts
-			(xy 177.8 77.47) (xy 163.83 77.47)
+			(xy 238.76 96.52) (xy 238.76 110.49)
 		)
 		(stroke
@@
 	(wire
 		(pts
-			(xy 238.76 96.52) (xy 238.76 110.49)
+			(xy 151.13 146.05) (xy 125.73 146.05)
 		)
 		(stroke
@@
 	(wire
 		(pts
-			(xy 151.13 146.05) (xy 125.73 146.05)
+			(xy 33.02 148.59) (xy 62.23 148.59)
 		)
 		(stroke
@@
 	(wire
 		(pts
-			(xy 161.29 80.01) (xy 161.29 36.83)
+			(xy 163.83 127) (xy 163.83 119.38)
 		)
 		(stroke
@@
 	(wire
 		(pts
-			(xy 163.83 127) (xy 163.83 119.38)
+			(xy 143.51 85.09) (xy 177.8 85.09)
 		)
 		(stroke
@@
 	(wire
 		(pts
-			(xy 143.51 85.09) (xy 177.8 85.09)
+			(xy 107.95 110.49) (xy 107.95 120.65)
 		)
 		(stroke
@@
 	(wire
 		(pts
-			(xy 107.95 110.49) (xy 107.95 120.65)
+			(xy 153.67 105.41) (xy 165.1 105.41)
 		)
 		(stroke
@@
 	(wire
 		(pts
-			(xy 153.67 105.41) (xy 165.1 105.41)
+			(xy 130.81 40.64) (xy 148.59 40.64)
 		)
 		(stroke
@@
 	(wire
 		(pts
-			(xy 130.81 40.64) (xy 148.59 40.64)
+			(xy 177.8 80.01) (xy 163.83 80.01)
 		)
 		(stroke
@@
 	(wire
 		(pts
-			(xy 227.33 115.57) (xy 227.33 119.38)
+			(xy 163.83 80.01) (xy 163.83 36.83)
 		)
 		(stroke
@@
 	(wire
 		(pts
-			(xy 33.02 146.05) (xy 35.56 146.05)
+			(xy 227.33 115.57) (xy 227.33 119.38)
 		)
 		(stroke
@@
 	(wire
 		(pts
-			(xy 165.1 107.95) (xy 158.75 107.95)
+			(xy 161.29 77.47) (xy 177.8 77.47)
 		)
 		(stroke
@@
 	(wire
 		(pts
-			(xy 238.76 111.76) (xy 238.76 114.3)
+			(xy 161.29 36.83) (xy 161.29 77.47)
 		)
 		(stroke
@@
 	(wire
 		(pts
-			(xy 33.02 148.59) (xy 62.23 148.59)
+			(xy 165.1 107.95) (xy 158.75 107.95)
+		)
+		(stroke
+			(width 0)
+			(type default)
+		)
+	)
+	(wire
+		(pts
+			(xy 238.76 111.76) (xy 238.76 114.3)
 		)
 		(stroke
@@
 	(wire
 		(pts
-			(xy 163.83 77.47) (xy 163.83 36.83)
-		)
-		(stroke
-			(width 0)
-			(type default)
-		)
-	)
-	(wire
-		(pts
 			(xy 57.15 143.51) (xy 57.15 138.43)
 		)
@@
 			)
 		)
-		(property "Footprint" "Capacitor_THT:CP_Radial_D8.0mm_P3.50mm"
+		(property "Footprint" "Capacitor_THT:CP_Radial_D7.5mm_P2.50mm"
 			(at 126.6952 146.05 0)
 			(effects
@@
 	(symbol
 		(lib_id "Connector_Generic:Conn_01x02")
-		(at 27.94 148.59 180)
+		(at 27.94 146.05 0)
+		(mirror y)
 		(unit 1)
 		(exclude_from_sim no)
@@
 		(dnp no)
 		(property "Reference" "J6"
-			(at 25.4 148.5901 0)
+			(at 25.4 146.0499 0)
 			(effects
 				(font
@@
 		)
 		(property "Value" "Photo Cel"
-			(at 25.4 146.0501 0)
+			(at 25.4 148.5899 0)
 			(effects
 				(font
@@
 			)
 		)
-		(property "Footprint" "PcbLibrary:Molex_SL_171971-0002_1x02_P2.54mm_Vertical_b"
-			(at 27.94 148.59 0)
+		(property "Footprint" "PcbLibrary:BorneBatSolar"
+			(at 27.94 146.05 0)
 			(effects
 				(font
@@
 		)
 		(property "Datasheet" "~"
-			(at 27.94 148.59 0)
+			(at 27.94 146.05 0)
 			(effects
 				(font
@@
 		)
 		(property "Description" "Generic connector, single row, 01x02, script generated (kicad-library-utils/schlib/autogen/connector/)"
-			(at 27.94 148.59 0)
+			(at 27.94 146.05 0)
 			(effects
 				(font
@@
 			)
 		)
-		(property "Footprint" "PcbLibrary:switch_3p_2mm_e_2.54mm"
+		(property "Footprint" "PcbLibrary:switch_3p_2.54mm_on_off"
 			(at 52.07 138.43 0)
 			(effects
@@
 			)
 		)
-		(property "Footprint" "PcbLibrary:switch_3p_2mm_e_2.54mm"
+		(property "Footprint" "PcbLibrary:switch_3p_2.54mm_on_off"
 			(at 139.7 134.62 0)
 			(effects
@@
 			)
 		)
-		(property "Footprint" "PcbLibrary:switch_3p_2mm_e_2.54mm"
+		(property "Footprint" "PcbLibrary:switch_3p_2.54mm_on_off"
 			(at 113.03 115.57 0)
 			(effects
@@
 			)
 		)
-		(property "Footprint" "Capacitor_THT:CP_Radial_D8.0mm_P3.50mm"
+		(property "Footprint" "Capacitor_THT:CP_Radial_D7.5mm_P2.50mm"
 			(at 215.5952 54.61 0)
 			(effects
@@
 			)
 		)
-		(property "Footprint" "Capacitor_THT:CP_Radial_D8.0mm_P3.50mm"
+		(property "Footprint" "Capacitor_THT:CP_Radial_D7.5mm_P2.50mm"
 			(at 190.1952 54.61 0)
 			(effects
